File: projects/PicoTracker1/PicoTracker1.sch (KiCad schematic (older format))
At the start: 10 parts, among them IC1 TPS61201, IC2 TPS61201, J1 Conn_01x02, M1 RF4463PRO, M2 UBLOX_NEO-6, U1 ATMEGA328-AU

Commit message: KiCad PicoTracker1 mid-development checkin
Parts:
- removed IC2: TPS61201, texas_S-PDSO-N10, symbol TPS61201
- removed J1: Conn_01x02, symbol Conn_01x02
- added BT1: Battery, Pin_Headers:Pin_Header_Straight_1x02_Pitch2.54mm, symbol Battery
- added C10, C7, C8, C9: .1uF, Capacitors_SMD:C_0603_HandSoldering, symbol C_Small
- added C4: 10uF, Capacitors_SMD:C_0603_HandSoldering, symbol C_Small
- added C5: 1uF, Capacitors_SMD:C_0603_HandSoldering, symbol C_Small
- added C6: 22uF, Capacitors_SMD:C_0603_HandSoldering, symbol C_Small
- added D1, D2, D3: LED_Small, LEDs:LED_0603_HandSoldering, symbol LED_Small
- added GPS_ANT1, GPS_GND1, RF_ANT1, RF_GND1: Conn_01x01, Measurement_Points:Measurement_Point_Square-SMD-Pad_Big, symbol Conn_01x01
- added GPS_SERIAL_TAP1, SERIAL1: Conn_01x02, Pin_Headers:Pin_Header_Straight_1x02_Pitch2.54mm, symbol Conn_01x02
- added L2: 2.2uH, Inductors_SMD:L_0603_HandSoldering, symbol L_Small
- added R1: 10k, Resistors_SMD:R_0603_HandSoldering, symbol R_Small
- added R2, R3, R4: 220, Resistors_SMD:R_0603_HandSoldering, symbol R_Small
- added REG_3V3_GPS1: TPS61201, CustomFootprintLibrary:texas-S-PDSO-N10, symbol TPS61201
- added SPI_PROG_HDR1: Conn_02x03_Odd_Even, Pin_Headers:Pin_Header_Straight_2x03_Pitch2.54mm, symbol Conn_02x03_Odd_Even
- C1, C2, C3: footprint (none) -> Capacitors_SMD:C_0603_HandSoldering
- L1: footprint (none) -> Inductors_SMD:L_0603_HandSoldering
- M1: footprint RF4436PRO_STD_BOARD -> CustomFootprintLibrary:RF4436PRO-STD_BOARD
- M2: footprint Ava_UBLOX_NEO-6P -> CustomFootprintLibrary:UBLOX_NEO-6
- REG_3V3_BOARD1: renamed from IC1; footprint texas_S-PDSO-N10 -> CustomFootprintLibrary:texas-S-PDSO-N10
Connections:
- net GND: now also M1.1 (GND), M1.12 (GND), M1.14 (GND), M2.10_G (10_GND), M2.12_G (12_GND), M2.13_G (13_GND), M2.24_G (24_GND), BT1.2 (-), C10.1, C4.2, C5.2, C6.2, C7.2, C8.2, C9.2, D1.1 (K), D2.1 (K), D3.1 (K), GPS_GND1.1 (Pin_1), REG_3V3_GPS1.4 (PGND), REG_3V3_GPS1.9 (GND), REG_3V3_GPS1.PP, REG_3V3_GPS1.PP@1 (PP), REG_3V3_GPS1.PP@2 (PP), RF_GND1.1 (Pin_1), SPI_PROG_HDR1.6 (Pin_6)
- net VBATT: now also BT1.1 (+), C4.1, L2.1, REG_3V3_GPS1.5 (VIN), REG_3V3_GPS1.7 (UVLO), REG_3V3_GPS1.8 (PS), SPI_PROG_HDR1.2 (Pin_2)
- net VCC: now also M1.5 (VCC), U1.18 (AVCC), U1.20 (AREF), U1.4 (VCC), U1.6 (VCC), C7.1, C9.1, R1.2
- net RF_SIGNAL: now reaches U1.1 ((PCINT19/OC2B/INT1)PD3)
- net RF_SIGNAL: now also M1.3 (GPIO0)
- net at U1.10 ((PCINT22/OC0A/AIN0)PD6): now also R3.2
- net at U1.11 ((PCINT23/AIN1)PD7): now also R2.2
- net RF_SHUTDOWN: now reaches U1.12 ((PCINT0/CLKO/ICP1)PB0)
- net RF_SHUTDOWN: now also M1.11 (SDN)
- net SPI_MOSI: now reaches U1.15 ((PCINT3/OC2A/MOSI)PB3)
- net SPI_MOSI: now also M1.7 (SDI), SPI_PROG_HDR1.4 (Pin_4)
- net SPI_MISO: now reaches U1.16 ((PCINT4/MISO)PB4)
- net SPI_MISO: now also M1.6 (SDO), SPI_PROG_HDR1.1 (Pin_1)
- net SPI_SCK: now reaches U1.17 ((PCINT5/SCK)PB5)
- net SPI_SCK: now also M1.8 (SCLK), SPI_PROG_HDR1.3 (Pin_3)
- net GPS_SER_OUT: now reaches U1.23 ((PCINT8/ADC0)PC0)
- net GPS_SER_OUT: now also M2.20_T (20_TXD1), GPS_SERIAL_TAP1.1 (Pin_1)
- net GPS_SER_IN: now reaches U1.24 ((PCINT9/ADC1)PC1)
- net GPS_SER_IN: now also M2.21_R (21_RXD1), GPS_SERIAL_TAP1.2 (Pin_2)
- net SPI_SS_RF: now reaches U1.25 ((PCINT10/ADC2)PC2)
- net SPI_SS_RF: now also M1.9 (NSEL)
- net GPS_ENABLE: now reaches U1.26 ((PCINT11/ADC3)PC3)
- net GPS_ENABLE: now also REG_3V3_GPS1.6 (EN)
- net SPI_RESET: now reaches U1.29 ((PCINT14/~RESET~)PC6)
- net SPI_RESET: now also R1.1, SPI_PROG_HDR1.5 (Pin_5)
- net at U1.30 ((PCINT16/RXD)PD0): now also SERIAL1.1 (Pin_1)
- net at U1.31 ((PCINT17/TXD)PD1): now also SERIAL1.2 (Pin_2)
- net at U1.9 ((PCINT21/OC0B/T1)PD5): now also R4.2
- net at M1.13 (ANT): now also RF_ANT1.1 (Pin_1)
- net at M2.11_R (11_RF_IN): now also GPS_ANT1.1 (Pin_1)
- net GPS_VCC: now reaches M2.22_V (22_V_BCKP)
- net GPS_VCC: now also M2.23_V (23_VCC), M2.7_VD (7_VDDUSB), M2.9_VC (9_VCC_RF), C10.2, C6.1, C8.1, REG_3V3_GPS1.10 (FB), REG_3V3_GPS1.2 (VOUT)
- new net: C5.1, REG_3V3_GPS1.1 (VAUX)
- new net: L2.2, REG_3V3_GPS1.3 (L)
- new net: D3.2 (A), R4.1
- new net: D2.2 (A), R3.1
- new net: D1.2 (A), R2.1
- no-connect marks 0 -> 26
Other:
- moved on the sheet: C1, C2, C3, L1, REG_3V3_BOARD1, U1
