File: projects/PicoTracker1/PicoTracker1.kicad_pcb (KiCad board)
At the start: 2 copper layers, 10 parts, among them IC1 TPS61201, IC2 TPS61201, J1 Conn_01x02, M1 RF4463PRO, M2 UBLOX_NEO-6, U1 ATMEGA328-AU

Commit message: KiCad PicoTracker1 mid-development checkin
Parts:
- removed IC1, IC2: TPS61201, CustomFootprintLibrary:texas-S-PDSO-N10
- removed J1: Conn_01x02, Pin_Headers:Pin_Header_Straight_1x02_Pitch1.27mm
- added BT1: Battery, Pin_Headers:Pin_Header_Straight_1x02_Pitch2.54mm, F.Cu at (209.6, 194.3)
- added C10: .1uF, Capacitors_SMD:C_0603_HandSoldering, F.Cu at (232.4, 187.3)
- added C4: 10uF, Capacitors_SMD:C_0603_HandSoldering, F.Cu at (217.8, 193.4)
- added C5: 1uF, Capacitors_SMD:C_0603_HandSoldering, F.Cu at (226.7, 193.4)
- added C6: 22uF, Capacitors_SMD:C_0603_HandSoldering, F.Cu at (224.5, 188.0)
- added C7: .1uF, Capacitors_SMD:C_0603_HandSoldering, F.Cu at (215.3, 171.4)
- added C8: .1uF, Capacitors_SMD:C_0603_HandSoldering, F.Cu at (228.6, 187.3)
- added C9: .1uF, Capacitors_SMD:C_0603_HandSoldering, F.Cu at (200.0, 175.3)
- added D1: LED_Small, LEDs:LED_0603_HandSoldering, F.Cu at (188.8, 167.6)
- added D2: LED_Small, LEDs:LED_0603_HandSoldering, F.Cu at (208.3, 167.6)
- added D3: LED_Small, LEDs:LED_0603_HandSoldering, F.Cu at (229.2, 169.5)
- added GPS_ANT1: Conn_01x01, Measurement_Points:Measurement_Point_Square-SMD-Pad_Big, F.Cu at (219.7, 168.9)
- added GPS_GND1: Conn_01x01, Measurement_Points:Measurement_Point_Square-SMD-Pad_Big, F.Cu at (224.2, 168.9)
- added GPS_SERIAL_TAP1: Conn_01x02, Pin_Headers:Pin_Header_Straight_1x02_Pitch2.54mm, F.Cu at (232.4, 191.8)
- added L2: 2.2uH, Inductors_SMD:L_0603_HandSoldering, F.Cu at (219.5, 188.0)
- added R1: 10k, Resistors_SMD:R_0603_HandSoldering, F.Cu at (198.6, 167.6)
- added R2: 220, Resistors_SMD:R_0603_HandSoldering, F.Cu at (192.9, 167.6)
- added R3: 220, Resistors_SMD:R_0603_HandSoldering, F.Cu at (203.8, 167.6)
- added R4: 220, Resistors_SMD:R_0603_HandSoldering, F.Cu at (229.2, 167.6)
- added REG_3V3_BOARD1: TPS61201, CustomFootprintLibrary:texas-S-PDSO-N10, F.Cu at (194.3, 193.3)
- added REG_3V3_GPS1: TPS61201, CustomFootprintLibrary:texas-S-PDSO-N10, F.Cu at (222.9, 193.0)
- added RF_ANT1: Conn_01x01, Measurement_Points:Measurement_Point_Square-SMD-Pad_Big, F.Cu at (181.0, 188.6)
- added RF_GND1: Conn_01x01, Measurement_Points:Measurement_Point_Square-SMD-Pad_Big, F.Cu at (185.4, 188.6)
- added SERIAL1: Conn_01x02, Pin_Headers:Pin_Header_Straight_1x02_Pitch2.54mm, F.Cu at (182.9, 193.0)
- added SPI_PROG_HDR1: Conn_02x03_Odd_Even, Pin_Headers:Pin_Header_Straight_2x03_Pitch2.54mm, F.Cu at (210.8, 186.7)
- moved M1 125.9 mm to (189.2, 177.8), turned to 180 degrees
- moved M2 117.3 mm to (224.8, 179.1), turned to 90 degrees
- moved C1 114.0 mm to (189.5, 193.7), turned to 90 degrees
- moved C3 108.8 mm to (196.2, 188.6)
- moved C2 107.1 mm to (198.1, 193.4), turned to 270 degrees
- moved L1 101.2 mm to (191.1, 188.6)
- moved U1 82.6 mm to (208.3, 176.5)
Connections:
- M2 pad 10_G: Net-(M2-Pad10_G) -> GND
- M2 pad 12_G: Net-(M2-Pad12_G) -> GND
- M2 pad 13_G: Net-(M2-Pad13_G) -> GND
- M2 pad 14_M: Net-(M2-Pad14_M) -> (no net)
- M2 pad 15_M: Net-(M2-Pad15_M) -> (no net)
- M2 pad 16_C: Net-(M2-Pad16_C) -> (no net)
- M2 pad 17_R: Net-(M2-Pad17_R) -> (no net)
- M2 pad 18_S: Net-(M2-Pad18_S) -> (no net)
- M2 pad 19_S: Net-(M2-Pad19_S) -> (no net)
- M2 pad 1_RE: Net-(M2-Pad1_RE) -> (no net)
- M2 pad 20_T: Net-(M2-Pad20_T) -> GPS_SER_OUT
- M2 pad 21_R: Net-(M2-Pad21_R) -> GPS_SER_IN
- M2 pad 22_V: Net-(M2-Pad22_V) -> GPS_VCC
- M2 pad 23_V: Net-(M2-Pad23_V) -> GPS_VCC
- M2 pad 24_G: Net-(M2-Pad24_G) -> GND
- M2 pad 2_SS: Net-(M2-Pad2_SS) -> (no net)
- M2 pad 3_TI: Net-(M2-Pad3_TI) -> (no net)
- M2 pad 4_EX: Net-(M2-Pad4_EX) -> (no net)
- M2 pad 5_US: Net-(M2-Pad5_US) -> (no net)
- M2 pad 6_US: Net-(M2-Pad6_US) -> (no net)
- M2 pad 7_VD: Net-(M2-Pad7_VD) -> GPS_VCC
- M2 pad 8_RE: Net-(M2-Pad8_RE) -> (no net)
- M2 pad 9_VC: Net-(M2-Pad9_VC) -> GPS_VCC
- U1 pad 1: Net-(U1-Pad1) -> RF_SIGNAL
- U1 pad 12: Net-(U1-Pad12) -> RF_SHUTDOWN
- U1 pad 13: Net-(U1-Pad13) -> (no net)
- U1 pad 14: Net-(U1-Pad14) -> (no net)
- U1 pad 15: Net-(U1-Pad15) -> SPI_MOSI
- U1 pad 16: Net-(U1-Pad16) -> SPI_MISO
- U1 pad 17: Net-(U1-Pad17) -> SPI_SCK
- U1 pad 18: Net-(U1-Pad18) -> VCC
- U1 pad 19: Net-(U1-Pad19) -> (no net)
- U1 pad 2: Net-(U1-Pad2) -> (no net)
- U1 pad 20: Net-(U1-Pad20) -> VCC
- U1 pad 22: Net-(U1-Pad22) -> (no net)
- U1 pad 23: Net-(U1-Pad23) -> GPS_SER_OUT
- U1 pad 24: Net-(U1-Pad24) -> GPS_SER_IN
- U1 pad 25: Net-(U1-Pad25) -> SPI_SS_RF
- U1 pad 26: Net-(U1-Pad26) -> GPS_ENABLE
- U1 pad 27: Net-(U1-Pad27) -> (no net)
- U1 pad 28: Net-(U1-Pad28) -> (no net)
- U1 pad 29: Net-(U1-Pad29) -> SPI_RESET
- U1 pad 32: Net-(U1-Pad32) -> (no net)
- U1 pad 4: Net-(U1-Pad4) -> VCC
- U1 pad 6: Net-(U1-Pad6) -> VCC
- U1 pad 7: Net-(U1-Pad7) -> (no net)
- U1 pad 8: Net-(U1-Pad8) -> (no net)
Routing:
- net VCC: track 0.00 -> 107.4 mm, vias 0 -> 6
- net VBATT: track 0.00 -> 72.9 mm
- net GPS_VCC: track 0.00 -> 63.4 mm, vias 0 -> 3
- net Net-(SERIAL1-Pad2): track 0.00 -> 49.0 mm, vias 0 -> 4
- net Net-(SERIAL1-Pad1): track 0.00 -> 48.5 mm, vias 0 -> 4
- net SPI_SCK: track 0.00 -> 45.3 mm
- net Net-(R4-Pad2): track 0.00 -> 41.4 mm, vias 0 -> 2
- net GPS_ENABLE: track 0.00 -> 39.7 mm, vias 0 -> 2
- net Net-(R2-Pad2): track 0.00 -> 38.5 mm, vias 0 -> 4
- net GPS_SER_IN: track 0.00 -> 34.9 mm, vias 0 -> 2
- net SPI_MOSI: track 0.00 -> 34.4 mm, vias 0 -> 2
- net SPI_MISO: track 0.00 -> 33.6 mm, vias 0 -> 2
- net GPS_SER_OUT: track 0.00 -> 31.7 mm, vias 0 -> 2
- net SPI_RESET: track 0.00 -> 30.6 mm, vias 0 -> 3
- net RF_SHUTDOWN: track 0.00 -> 22.3 mm, vias 0 -> 2
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- added copper zone on B.Cu, net GND
- added copper zone on F.Cu, net GND
Other:
- board outline added: 58.4 x 32.4 mm
- rule pad_to_mask_clearance: 0.2 -> 0.0508

Commit message: KiCad PicoTracker1 pcb done
Parts:
- moved R1 24.1 mm to (208.9, 189.4), turned to 270 degrees
- moved SERIAL1 20.9 mm to (203.2, 188.0)
- moved R4 20.8 mm to (209.1, 172.7)
- moved D3 20.2 mm to (209.1, 170.8)
- moved GPS_SERIAL_TAP1 19.1 mm to (213.4, 190.5), turned to 180 degrees
- moved SPI_PROG_HDR1 15.7 mm to (197.5, 178.4), turned to 0 degrees
- moved C8 14.9 mm to (214.0, 184.5), turned to 270 degrees
- moved C10 13.8 mm to (230.5, 173.7), turned to 270 degrees
- moved D1 11.9 mm to (200.2, 170.8)
- moved R2 8.91 mm to (200.2, 172.7), turned to 0 degrees
- moved C7 8.17 mm to (213.4, 179.4), turned to 270 degrees
- moved R3 5.14 mm to (204.6, 172.7)
- moved RF_ANT1 5.08 mm to (175.9, 188.6)
- moved RF_GND1 5.08 mm to (180.3, 188.6)
- moved D2 4.83 mm to (204.6, 170.8)
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Routing:
- net GND: track 15.5 -> 61.6 mm, vias 0 -> 3
- net VBATT: track 72.9 -> 109.9 mm, vias 0 -> 6
- net Net-(SERIAL1-Pad2): track 49.0 -> 12.7 mm, vias 4 -> 1
- net Net-(SERIAL1-Pad1): track 48.5 -> 12.3 mm, vias 4 -> 1
- net Net-(R4-Pad2): track 41.4 -> 6.06 mm
- net Net-(R2-Pad2): track 38.5 -> 11.3 mm, vias 4 -> 2
- net VCC: track 107.4 -> 81.8 mm, vias 6 -> 2
- net SPI_SCK: track 45.3 -> 24.4 mm, vias 0 -> 2
- net RF_SIGNAL: track 14.2 -> 32.5 mm, vias 0 -> 2
- net SPI_SS_RF: track 17.3 -> 34.2 mm, vias 0 -> 2
- net SPI_MISO: track 33.6 -> 17.6 mm
- net Net-(R3-Pad2): track 18.4 -> 7.07 mm
- net GPS_SER_IN: track 34.9 -> 24.0 mm
- net SPI_RESET: track 30.6 -> 22.0 mm
- net GPS_SER_OUT: track 31.7 -> 39.4 mm
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Other:
- board size 58.4 x 32.4 mm -> 60.3 x 33.7 mm
- net class Default: clearance 0.2 -> 0.1524; trace_width 0.25 -> 0.1524; via_dia 0.6 -> 0.6858; via_drill 0.4 -> 0.3302
- rule trace_clearance: 0.2 -> 0.1524
- rule trace_min: 0.2 -> 0.1524
- rule via_min_drill: 0.3 -> 0.3302
- rule via_min_size: 0.4 -> 0.6858
- board text added: "2018-01-29 - PicoTracker1 - Rev 1"
- board text added: "Safe scientific experiment in Ham Radio (APRS) If found, please contact us! Douglas Malnati (KD2KDD) Mark Malnati (KN4IUD) douglas.malnati@gmail.com 201-993-6716"
