File: projects/EvilEye/EvilEye.kicad_pcb (KiCad board)
At the start: 2 copper layers, 85 parts, among them Q1 2N2219, Q2 2N2219, Q3 2N2219, Q4 2N2219, SW1 SW_SPDT, U1 CAP1188-1-CP-TR, U2 ATMEGA328P-AU

Commit message: KiCad EvilEye final
Parts:
- added G***: LOGO, CustomFootprintArtworkLibrary:border_ivy_copper, F.Cu at (250.7, 80.5)
- added G***: LOGO, CustomFootprintArtworkLibrary:border_ivy_copper, F.Cu at (191.0, 95.0)
- added REF**: Test_Point_Keystone_5019_Minature, Measurement_Points:Test_Point_Keystone_5019_Minature, B.Cu at (258.3, 112.5)
- added REF**: Test_Point_Keystone_5019_Minature, Measurement_Points:Test_Point_Keystone_5019_Minature, B.Cu at (182.9, 112.5)
- added svg2mod: G***, CustomFootprintArtworkLibrary:logo_dm_10x10mm, B.Cu at (186.7, 66.3)
Routing:
- net GND: track 106.8 -> 113.8 mm
- net Net-(D1-Pad1): track 104.8 -> 99.8 mm
- net ROW8: track 158.1 -> 161.0 mm
- net COL1: track 43.5 -> 45.8 mm
- net VCC: track 60.2 -> 58.2 mm
- net SPI_SCK: track 157.8 -> 156.5 mm
- net ROW10: track 165.1 -> 163.9 mm
- net Net-(Q3-Pad2): track 28.2 -> 27.3 mm
- net Net-(D29-Pad1): track 157.7 -> 156.8 mm
- net Net-(SENSE1-Pad1): track 22.3 -> 21.7 mm
Other:
- board outline added: 81.3 x 55.6 mm

Commit message: KiCad EvilEye twaeaks and artifacts of upgrading to 5.0
Other:
- board text added: "wrong footprint for transistors (flipped on back necessary) also hookup for cap1188 is wrong"
Changed lines of the file:
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@@
-(kicad_pcb (version 4) (host pcbnew 4.0.7)
+(kicad_pcb (version 20171130) (host pcbnew "(5.0.1)-rc2")
   (general
-    (links 0)
-    (no_connects 0)
-    (area 180.264999 59.868999 261.695001 115.645001)
     (thickness 1.6)
-    (drawings 14)
+    (drawings 15)
     (tracks 1888)
     (zones 0)
@@
     (pad_drill 0)
     (pad_to_mask_clearance 0.2)
+    (solder_mask_min_width 0.25)
     (aux_axis_origin 0 0)
     (visible_elements 7FFFFFFF)
@@
       (layerselection 0x00030_80000001)
       (usegerberextensions false)
+      (usegerberattributes false)
+      (usegerberadvancedattributes false)
+      (creategerberjobfile false)
       (excludeedgelayer true)
       (linewidth 0.100000)
@@
       (hpglpennumber 1)
       (hpglpenspeed 20)
-      (hpglpendiameter 15)
-      (hpglpenoverlay 2)
+      (hpglpendiameter 15.000000)
       (psnegative false)
       (psa4output false)
@@
     (at 250.698 80.518 180)
     (fp_text reference G*** (at 0 0 180) (layer F.Mask) hide
-      (effects (font (thickness 0.3)))
+      (effects (font (size 1.524 1.524) (thickness 0.3)))
     )
     (fp_text value LOGO (at 0.75 0 180) (layer F.Mask) hide
-      (effects (font (thickness 0.3)))
+      (effects (font (size 1.524 1.524) (thickness 0.3)))
     )
     (fp_poly (pts (xy 7.206263 18.215963) (xy 7.271571 18.433073) (xy 7.281593 18.739761) (xy 7.241648 19.067485)
@@
     (attr smd)
     (fp_text reference svg2mod (at 0 8.056576 180) (layer B.SilkS) hide
-      (effects (font (thickness 0.3048)) (justify mirror))
+      (effects (font (size 1.524 1.524) (thickness 0.3048)) (justify mirror))
     )
     (fp_text value G*** (at 0 -8.056576 180) (layer B.SilkS) hide
-      (effects (font (thickness 0.3048)) (justify mirror))
+      (effects (font (size 1.524 1.524) (thickness 0.3048)) (justify mirror))
     )
     (fp_poly (pts (xy -1.980338 2.075986) (xy -2.094814 0.823808) (xy -1.832128 0.741127) (xy -1.598937 0.586581)
@@
     (at 191.008 94.996)
     (fp_text reference G*** (at 0 0) (layer F.Mask) hide
-      (effects (font (thickness 0.3)))
+      (effects (font (size 1.524 1.524) (thickness 0.3)))
     )
     (fp_text value LOGO (at 0.75 0) (layer F.Mask) hide
-      (effects (font (thickness 0.3)))
+      (effects (font (size 1.524 1.524) (thickness 0.3)))
     )
     (fp_poly (pts (xy 7.206263 18.215963) (xy 7.271571 18.433073) (xy 7.281593 18.739761) (xy 7.241648 19.067485)
@@
     (pad 1 smd rect (at 0 0 270) (size 3.8 2) (layers B.Cu B.Paste B.Mask))
   )
+  (gr_text "wrong footprint for transistors (flipped on back necessary)\nalso hookup for cap1188 is wrong" (at 221.234 55.118) (layer B.SilkS)
+    (effects (font (size 1.5 1.5) (thickness 0.3)) (justify mirror))
+  )
   (gr_line (start 180.34 59.944) (end 180.34 115.57) (layer Edge.Cuts) (width 0.15))
