File: projects/PicoTrackerWSPR1Rev2/PicoTrackerWSPR1Rev2.sch (KiCad schematic (older format))
At the start: 51 parts, among them J1 Conn_01x02, M1 SIP32431DR3-T1GE3, M2 SIP32431DR3-T1GE3, M3 UBLOX_NEO-6, M4 SI5351A, U1 ATMEGA328P-AU, Y1 CRYSTAL_ABM8G

Commit message: KiCad PicoTrackerWSPR1Rev2 complete
Parts:
- added CONN25: GND_TAP, Socket_Strips:Socket_Strip_Straight_1x01_Pitch2.54mm, symbol conn:Conn_01x01
- CONN3: value VCC_INPUT -> BATT_INPUT
- CONN7: value VCC_TAP -> BATT_TAP
- CONN8: value GND_TAP -> VCC_TAP
Connections:
- net GND: now also CONN25.1 (Pin_1); no longer CONN8.1 (Pin_1)
- net VBATT: now also CONN3.1 (Pin_1), CONN7.1 (Pin_1)
- net VCC: now also CONN8.1 (Pin_1); no longer CONN3.1 (Pin_1), CONN7.1 (Pin_1)
Other:
- moved on the sheet: CONN3, CONN4, CONN7
Changed lines of the file:
@@
 L conn:Conn_01x01 CONN7
 U 1 1 5AD5DC66
-P 7650 9050
-F 0 "CONN7" H 7650 9150 50  0000 C CNN
-F 1 "VCC_TAP" H 7650 8950 50  0000 C CNN
-F 2 "Socket_Strips:Socket_Strip_Straight_1x01_Pitch2.54mm" H 7650 9050 50  0001 C CNN
-F 3 "" H 7650 9050 50  0001 C CNN
-	1    7650 9050
-	1    0    0    -1
-$EndComp
-Text GLabel 7450 9050 0    60   Input ~ 0
-VCC
+P 6950 9550
+F 0 "CONN7" H 6950 9650 50  0000 C CNN
+F 1 "BATT_TAP" H 6950 9450 50  0000 C CNN
+F 2 "Socket_Strips:Socket_Strip_Straight_1x01_Pitch2.54mm" H 6950 9550 50  0001 C CNN
+F 3 "" H 6950 9550 50  0001 C CNN
+	1    6950 9550
+	1    0    0    -1
+$EndComp
+Text GLabel 6750 9550 0    60   Input ~ 0
+VBATT
 NoConn ~ 8950 9800
 NoConn ~ 8950 10350
@@
 Connection ~ 13700 8800
 $Comp
-L conn:Conn_01x01 CONN8
-U 1 1 5C711443
-P 7650 9350
-F 0 "CONN8" H 7650 9450 50  0000 C CNN
-F 1 "GND_TAP" H 7650 9250 50  0000 C CNN
-F 2 "Socket_Strips:Socket_Strip_Straight_1x01_Pitch2.54mm" H 7650 9350 50  0001 C CNN
-F 3 "" H 7650 9350 50  0001 C CNN
-	1    7650 9350
-	1    0    0    -1
-$EndComp
-Text GLabel 7450 9350 0    60   Input ~ 0
-GND
-$Comp
 L conn:Conn_01x01 CONN3
 U 1 1 5C713AD8
-P 6950 9050
-F 0 "CONN3" H 6950 9150 50  0000 C CNN
-F 1 "VCC_INPUT" H 6950 8950 50  0000 C CNN
-F 2 "Socket_Strips:Socket_Strip_Straight_1x01_Pitch2.54mm" H 6950 9050 50  0001 C CNN
-F 3 "" H 6950 9050 50  0001 C CNN
-	1    6950 9050
-	1    0    0    -1
-$EndComp
-Text GLabel 6750 9050 0    60   Input ~ 0
-VCC
+P 6950 8700
+F 0 "CONN3" H 6950 8800 50  0000 C CNN
+F 1 "BATT_INPUT" H 6950 8600 50  0000 C CNN
+F 2 "Socket_Strips:Socket_Strip_Straight_1x01_Pitch2.54mm" H 6950 8700 50  0001 C CNN
+F 3 "" H 6950 8700 50  0001 C CNN
+	1    6950 8700
+	1    0    0    -1
+$EndComp
+Text GLabel 6750 8700 0    60   Input ~ 0
+VBATT
 $Comp
 L conn:Conn_01x01 CONN4
 U 1 1 5C713ADF
-P 6950 9350
-F 0 "CONN4" H 6950 9450 50  0000 C CNN
-F 1 "GND_INPUT" H 6950 9250 50  0000 C CNN
-F 2 "Socket_Strips:Socket_Strip_Straight_1x01_Pitch2.54mm" H 6950 9350 50  0001 C CNN
-F 3 "" H 6950 9350 50  0001 C CNN
-	1    6950 9350
-	1    0    0    -1
-$EndComp
-Text GLabel 6750 9350 0    60   Input ~ 0
+P 6950 9000
+F 0 "CONN4" H 6950 9100 50  0000 C CNN
+F 1 "GND_INPUT" H 6950 8900 50  0000 C CNN
+F 2 "Socket_Strips:Socket_Strip_Straight_1x01_Pitch2.54mm" H 6950 9000 50  0001 C CNN
+F 3 "" H 6950 9000 50  0001 C CNN
+	1    6950 9000
+	1    0    0    -1
+$EndComp
+Text GLabel 6750 9000 0    60   Input ~ 0
 GND
 Wire Notes Line
@@
 Text Notes 10750 2650 0    50   ~ 0
 Cut Trace for\nmisbehaving modules
+$Comp
+L conn:Conn_01x01 CONN8
+U 1 1 5C70A805
+P 6950 9850
+F 0 "CONN8" H 6950 9950 50  0000 C CNN
+F 1 "VCC_TAP" H 6950 9750 50  0000 C CNN
+F 2 "Socket_Strips:Socket_Strip_Straight_1x01_Pitch2.54mm" H 6950 9850 50  0001 C CNN
+F 3 "" H 6950 9850 50  0001 C CNN
+	1    6950 9850
+	1    0    0    -1
+$EndComp
+Text GLabel 6750 9850 0    60   Input ~ 0
+VCC
+$Comp
+L conn:Conn_01x01 CONN25
+U 1 1 5C70A80C
+P 6950 10150
+F 0 "CONN25" H 6950 10250 50  0000 C CNN
+F 1 "GND_TAP" H 6950 10050 50  0000 C CNN
+F 2 "Socket_Strips:Socket_Strip_Straight_1x01_Pitch2.54mm" H 6950 10150 50  0001 C CNN
+F 3 "" H 6950 10150 50  0001 C CNN
+	1    6950 10150
+	1    0    0    -1
+$EndComp
+Text GLabel 6750 10150 0    60   Input ~ 0
+GND
 $EndSCHEMATC

Commit message: KiCad PicoTrackerWSPR1Rev2 added forgotten battery sense voltage divider
Parts:
- added R7, R8: 1M, Resistors_SMD:R_0603_HandSoldering, symbol Device:R_Small
Connections:
- net GND: now also R8.1
- net VBATT: now also R7.2; no longer U1.26 ((PCINT11/ADC3)PC3)
- new net VBATT_SENSE: R7.1, R8.2, U1.26 ((PCINT11/ADC3)PC3)
Changed lines of the file:
@@
 	12400 3250 12500 3250
 Text GLabel 3950 6250 2    60   Input ~ 0
-VBATT
+VBATT_SENSE
 Text Notes 7700 7450 0    50   ~ 0
 Break-off Parts
@@
 Text GLabel 7000 3950 2    50   Input ~ 0
 VBATT
-Wire Notes Line
-	5700 3500 5700 4650
-Wire Notes Line
-	5700 4650 7450 4650
-Wire Notes Line
-	7450 4650 7450 3500
-Wire Notes Line
-	7450 3500 5700 3500
 $Comp
 L CustomSchematicLibrary:ATMEGA328P-AU U1
@@
 Text GLabel 6750 10150 0    60   Input ~ 0
 GND
+$Comp
+L Device:R_Small R7
+U 1 1 5C74C6E2
+P 7500 4000
+F 0 "R7" H 7530 4020 50  0000 L CNN
+F 1 "1M" H 7530 3960 50  0000 L CNN
+F 2 "Resistors_SMD:R_0603_HandSoldering" H 7500 4000 50  0001 C CNN
+F 3 "" H 7500 4000 50  0001 C CNN
+	1    7500 4000
+	-1   0    0    1
+$EndComp
+$Comp
+L Device:R_Small R8
+U 1 1 5C74CD20
+P 7500 4400
+F 0 "R8" H 7530 4420 50  0000 L CNN
+F 1 "1M" H 7530 4360 50  0000 L CNN
+F 2 "Resistors_SMD:R_0603_HandSoldering" H 7500 4400 50  0001 C CNN
+F 3 "" H 7500 4400 50  0001 C CNN
+	1    7500 4400
+	-1   0    0    1
+$EndComp
+$Comp
+L power:GND #PWR06
+U 1 1 5C74CDAA
+P 7500 4650
+F 0 "#PWR06" H 7500 4400 50  0001 C CNN
+F 1 "GND" H 7500 4500 50  0000 C CNN
+F 2 "" H 7500 4650 50  0001 C CNN
+F 3 "" H 7500 4650 50  0001 C CNN
+	1    7500 4650
+	1    0    0    -1
+$EndComp
+Text GLabel 7500 3700 2    50   Input ~ 0
+VBATT
+Wire Wire Line
+	7500 3700 7500 3900
+Wire Wire Line
+	7500 4650 7500 4500
+Wire Wire Line
+	7500 4100 7500 4300
+Text GLabel 7500 4200 2    50   Input ~ 0
+VBATT_SENSE
+Wire Notes Line
+	5700 3500 5700 4900
+Wire Notes Line
+	5700 4900 8150 4900
+Wire Notes Line
+	8150 4900 8150 3500
+Wire Notes Line
+	8150 3500 5700 3500
 $EndSCHEMATC
