File: projects/ModuleSolarToStorageLTC3105/ModuleSolarToStorageLTC3105.sch (KiCad schematic (older format))
At the start: 10 parts, among them U1 LTC3105EMS-PBF

Commit message: KiCad ModuleSolarToStorageLTC3105 Rev2
Parts:
- removed C4: C_Small, Capacitors_SMD:C_0603_HandSoldering, symbol Device:C_Small
- removed GND_EXTERNAL1, GND_EXTERNAL2, VIN_EXTERNAL2, VOUT_EXTERNAL1: Conn_01x01_Female, Socket_Strips:Socket_Strip_Straight_1x01_Pitch2.54mm, symbol Connector:Conn_01x01_Female
- removed L1: L_Small, CustomFootprintLibrary:coilcraft-MSS5131-103, symbol Device:L_Small
- added C1: ??uF, Capacitors_SMD:C_0603_HandSoldering, symbol Device:C_Small
- added J1: VIN, Socket_Strips:Socket_Strip_Straight_1x01_Pitch2.54mm, symbol Connector:Conn_01x01_Female
- added J2, J5: GND, Socket_Strips:Socket_Strip_Straight_1x01_Pitch2.54mm, symbol Connector:Conn_01x01_Female
- added J3: VOUT, Socket_Strips:Socket_Strip_Straight_1x01_Pitch2.54mm, symbol Connector:Conn_01x01_Female
- added J4: LDO, Socket_Strips:Socket_Strip_Straight_1x01_Pitch2.54mm, symbol Connector:Conn_01x01_Female
- added L1: 10uH, CustomFootprintLibrary:coilcraft-MSS5131-103, symbol Device:L
- added R1, R2, R4, R5: R_Small, Resistors_SMD:R_0603_HandSoldering, symbol Device:R_Small
- C2: value C_Small -> 1uF
- C3: value C_Small -> ??uF; footprint Capacitors_SMD:C_0603_HandSoldering -> Capacitors_Tantalum_SMD:CP_Tantalum_Case-U_EIA-6032-15_Hand
Connections:
- net GND: now also C1.2, J2.1 (Pin_1), J5.1 (Pin_1), R2.2, R4.2, R5.2; no longer R3.2, U1.1 (FB), U1.3 (FBLDO)
- net VIN: now also C3.1, J1.1 (Pin_1), L1.2; no longer C2.1
- net VOUT: now also C1.1, J3.1 (Pin_1), R1.1; no longer C3.1
- net LDO: now reaches U1.2 (LDO)
- net LDO: now also R3.1, J4.1 (Pin_1)
- net AUX: no longer names the net of U1.12 (AUX)
- net AUX: now also C2.1
- net MPPC_PROGRAMMING: no longer names the net of U1.5 (MPPC)
- net MPPC_PROGRAMMING: now also R5.1; no longer R3.1
- net SW: no longer names the net of U1.9 (SW)
- net SW: now also L1.1
- new net: R1.2, R2.1, U1.1 (FB)
- new net: R3.2, R4.1, U1.3 (FBLDO)
- no-connect marks 4 -> 2
Other:
- note removed: "Board Input/Output"
- note removed: "Board Programming"
