File: projects/PicoTrackerWSPR1Rev4/PicoTrackerWSPR1Rev4.sch (KiCad schematic (older format))
At the start: 54 parts, among them J1 Conn_01x02, M1 SIP32431DR3-T1GE3, M2 SIP32431DR3-T1GE3, M3 UBLOX_NEO-6, M4 SI5351A, U1 ATMEGA328P-AU, Y1 CRYSTAL_ABM8G

Commit message: KiCad PicoTrackerWSPR1Rev4 done
Parts:
- removed Y1: CRYSTAL_ABM8G, CustomFootprintLibrary:ABM8G-25.000MHZ-B4Y-T, symbol CustomSchematicLibrary:CRYSTAL_ABM8G
- added R10: 68, Resistors_SMD:R_0603_HandSoldering, symbol Device:R
- added R11, R9: 100, Resistors_SMD:R_0603_HandSoldering, symbol Device:R
- added R5: R_Small, Resistors_SMD:R_0603_HandSoldering, symbol Device:R_Small
- added TCXO1, TCXO2: CRYSTAL_TCXO_3.2mmWidth_2.5mmHeight, CustomFootprintLibrary:CRYSTAL_3.2mmWidth_2.5mmHeight, symbol CustomSchematicLibrary:CRYSTAL_TCXO_3.2mmWidth_2.5mmHeight
- added TH1: PT100, CustomFootprintLibrary:PTS060301B100RP100, symbol Sensor_Temperature:PT100
Connections:
- net GND: now also R11.2, R9.2, TCXO1.2, TCXO2.2, TH1.1
- net SCL: now also R6.2
- net SIG_B: now also U1.32 ((PCINT18/INT0)PD2); no longer U1.25 ((PCINT10/ADC2)PC2)
- net SPI_RESET: now also R3.2; no longer R6.2
- net VCC: now also TCXO1.1, TCXO1.4; no longer J1.1 (Pin_1)
- net WSPR_VCC: now also TCXO2.1, TCXO2.4
- net at M4.2 (XA): now also R10.1, R11.1
- net at U1.7 ((PCINT6/XTAL1/TOSC1)PB6): now also TCXO1.3
- net TEMP_ENABLE: now reaches U1.9 ((PCINT21/OC0B/T1)PD5)
- net TEMP_ENABLE: now also R5.1
- net RESET renamed GPS_V_BCKP
- net GPS_V_BCKP: now also J1.1 (Pin_1); no longer R3.2
- new net: R10.2, R9.1, TCXO2.3
- new net VTEMP_SENSE: R5.2, TH1.2, U1.25 ((PCINT10/ADC2)PC2)
- no-connect marks 24 -> 22
Other:
- note added: "TCXO\n(not mandatory)\n(fuses dictate)"
- note added: "Temperature sensor"
- note removed: "SCL omitted purposefully.\nThe clockgen tries to power itself through\nthis when shut off.\nTested working without it."
- moved on the sheet: C1, C10, C11, C7, C8, C9, CONN1, CONN10, CONN11, CONN12, CONN13, CONN14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
