File: projects/PicoTrackerWSPR2Rev1/PicoTrackerWSPR2Rev1.kicad_pcb (KiCad board)
At the start: 2 copper layers, 42.9 x 29.5 mm, 48 parts, among them IC1 MCP9808, M4 SI5351A, U1 UBLOX_MAX-7, U2 SIP32431DNP3-T1GE4, U3 ATMEGA328P-MU

Commit message: PicoTrackerWSPR2Rev1 silkscreen
Other:
- board text added: "KD2KDD"
- board text added: "KN4IUD"
- board text added: "PicoTrackerWSPR2 Rev1 2020-03-16"
- board text added: "picoballoons.net"
Changed lines of the file:
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@@
   (general
     (thickness 1.6)
-    (drawings 30)
+    (drawings 34)
     (tracks 572)
     (zones 0)
@@
     (tags "Mesurement Point Square SMD Pad 3x3mm")
     (attr virtual)
-    (fp_text reference CONN26 (at 0 3 90) (layer B.SilkS)
+    (fp_text reference CONN26 (at 0 3 90) (layer B.SilkS) hide
       (effects (font (size 1 1) (thickness 0.15)) (justify mirror))
     )
@@
     (tags "Mesurement Point Square SMD Pad 3x3mm")
     (attr virtual)
-    (fp_text reference CONN1 (at 0 3 90) (layer B.SilkS)
+    (fp_text reference CONN1 (at 0 3 90) (layer B.SilkS) hide
       (effects (font (size 1 1) (thickness 0.15)) (justify mirror))
     )
@@
       (rotate (xyz 0 0 0))
     )
+  )
+  (gr_text KN4IUD (at 76.835 75.819 90) (layer B.SilkS)
+    (effects (font (size 0.8 0.8) (thickness 0.15)) (justify mirror))
+  )
+  (gr_text KD2KDD (at 76.835 69.596 90) (layer B.SilkS)
+    (effects (font (size 0.8 0.8) (thickness 0.15)) (justify mirror))
+  )
+  (gr_text picoballoons.net (at 74.168 72.644 90) (layer B.SilkS)
+    (effects (font (size 0.8 0.8) (thickness 0.15)) (justify mirror))
+  )
+  (gr_text "PicoTrackerWSPR2\nRev1\n2020-03-16" (at 113.03 75.692) (layer B.SilkS)
+    (effects (font (size 1 1) (thickness 0.15)) (justify left mirror))
   )
   (dimension 12.192 (width 0.15) (layer F.SilkS)
@@
   (segment (start 99.5905 67.118) (end 99.515499 67.042999) (width 0.25) (layer F.Cu) (net 1))
   (segment (start 99.5905 67.818) (end 99.5905 67.118) (width 0.25) (layer F.Cu) (net 1) (status 10))
-  (segment (start 86.816171 75.394571) (end 86.0878 74.6662) (width 0.25) (layer F.Cu) (net 13))
-  (segment (start 86.0878 74.6662) (end 84.9378 74.6662) (width 0.25) (layer F.Cu) (net 13) (status 20))
-  (segment (start 88.569705 75.016528) (end 88.191662 75.394571) (width 0.25) (layer F.Cu) (net 13) (status 10))
   (segment (start 86.897 67.818) (end 87.122 67.818) (width 0.25) (layer F.Cu) (net 2) (status 30))
   (segment (start 85.5488 69.1662) (end 86.897 67.818) (width 0.25) (layer F.Cu) (net 2) (status 30))
@@
   (segment (start 87.884 91.694) (end 88.605144 90.972856) (width 0.25) (layer B.Cu) (net 12))
   (segment (start 88.605144 90.972856) (end 88.605144 84.907018) (width 0.25) (layer B.Cu) (net 12))
+  (segment (start 86.816171 75.394571) (end 86.0878 74.6662) (width 0.25) (layer F.Cu) (net 13))
+  (segment (start 86.0878 74.6662) (end 84.9378 74.6662) (width 0.25) (layer F.Cu) (net 13) (status 20))
+  (segment (start 88.569705 75.016528) (end 88.191662 75.394571) (width 0.25) (layer F.Cu) (net 13) (status 10))
   (segment (start 87.419429 75.394571) (end 87.419429 75.307539) (width 0.25) (layer F.Cu) (net 13))
   (segment (start 87.419429 75.394571) (end 86.816171 75.394571) (width 0.25) (layer F.Cu) (net 13))
