File: projects/BreakoutGPSATGM336H/BreakoutGPSATGM336H.sch (KiCad schematic (older format))
At the start: 3 parts, among them J1 Conn_01x09_Female, J2 Conn_01x09_Female, U1 UBLOX_MAX-7

Commit message: BreakoutGPSATGM336H
Connections:
- net at U1.13 (NC): now also J1.6 (Pin_6)
- net at U1.15 (NC): now also J1.4 (Pin_4)
- net at U1.18 (NC): now also J1.1 (Pin_1)
- net at U1.7 (NC): now also J2.3 (Pin_3)
- no-connect marks 4 -> 0
Changed lines of the file:
@@
 	5000 4050 4800 4050
-Wire Wire Line
-	6000 4150 6100 4150
 Wire Wire Line
 	6200 4050 6000 4050
@@
 Wire Wire Line
 	6200 3350 6000 3350
-NoConn ~ 6200 3550
-NoConn ~ 4800 4150
-NoConn ~ 4800 3850
-NoConn ~ 4800 3650
 $Comp
 L power:PWR_FLAG #FLG04
@@
 	0    1    1    0
 $EndComp
-Connection ~ 6100 4150
-Wire Wire Line
-	6100 4150 6200 4150
 Text GLabel 6850 3850 0    50   Input ~ 0
 GND
@@
 Text GLabel 4950 3550 1    50   Input ~ 0
 GND
+Wire Wire Line
+	6000 4150 6200 4150
+Wire Wire Line
+	4800 3650 5000 3650
+Wire Wire Line
+	5000 3850 4800 3850
+Wire Wire Line
+	4800 4150 5000 4150
+Wire Wire Line
+	6000 3550 6200 3550
 $EndSCHEMATC
