File: projects/BikeLightComputer/BikeLightComputer.kicad_pcb (KiCad board)
At the start: 2 copper layers, 28 parts, among them IC1 MOSFET_SOT223_FQT13N06TF, IC2 MOSFET_SOT223_FQT13N06TF, IC3 MOSFET_SOT223_FQT13N06TF, IC4 REG_3V3_NCP1117ST33T3G, J1 Barrel_Jack_MountingPin, J10 Conn_01x01_Male, J11 Conn_01x01_Male, J12 Conn_01x01_Male, J13 Conn_01x01_Male, J14 Conn_01x01_Male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

Commit message: BikeLightComputer done
Parts:
- moved J10 55.6 mm to (172.7, 66.5), turned to 180 degrees
- moved J11 54.5 mm to (172.7, 69.1), turned to 180 degrees
- moved J12 54.0 mm to (172.7, 71.6), turned to 180 degrees
- moved J13 50.7 mm to (170.2, 66.5), turned to 180 degrees
- moved J14 49.5 mm to (170.2, 69.1), turned to 180 degrees
- moved J15 48.9 mm to (170.2, 71.6), turned to 180 degrees
- moved J2 38.8 mm to (172.7, 85.9)
- moved J16 27.4 mm to (160.0, 94.2)
- moved C3 24.2 mm to (158.8, 66.0), turned to 0 degrees
- moved C2 23.8 mm to (155.2, 66.0), turned to 0 degrees
- moved C5 23.7 mm to (150.9, 66.0), turned to 180 degrees
- moved J4 23.6 mm to (145.8, 89.9), turned to 270 degrees
- moved C6 23.5 mm to (146.3, 66.0), turned to 0 degrees
- moved C1 22.4 mm to (155.2, 67.8), turned to 0 degrees
- moved C4 21.9 mm to (158.7, 67.8), turned to 0 degrees
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Routing:
- net VCC: track 46.4 -> 101.0 mm, vias 1 -> 4
- net GND: track 0.00 -> 50.1 mm, vias 0 -> 7
- net SPI_MOSI: track 10.0 -> 55.0 mm, vias 1 -> 3
- net VOLTAGE_INPUT: track 30.3 -> 67.6 mm, vias 0 -> 3
- net SPI_MISO: track 8.56 -> 38.7 mm, vias 1 -> 3
- net SPI_RESET: track 0.00 -> 25.4 mm, vias 0 -> 1
- net AVR_SER_RX: track 0.00 -> 24.0 mm, vias 0 -> 3
- net AVR_SER_TX: track 0.00 -> 22.5 mm, vias 0 -> 3
- net SPI_SCK: track 12.5 -> 33.7 mm, vias 2 -> 3
- net AVR_PWM_BLUE: track 0.00 -> 17.5 mm, vias 0 -> 2
- net AVR_PWM_RED: track 0.00 -> 16.6 mm, vias 0 -> 2
- net Net-(J1-Pad1): track 19.1 -> 34.1 mm
- net RADIO_SDN: track 19.4 -> 6.42 mm, vias 3 -> 1
- net AVR_PWM_GREEN: track 0.00 -> 12.8 mm, vias 0 -> 2
- net RADIO_NIRQ: track 21.7 -> 9.17 mm
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- added copper zone on B.Cu, net GND
- added copper zone on F.Cu, net GND
Other:
- board outline added: 32.3 x 36.3 mm
- board text added: "12V"
- board text added: "12V GND"
- board text added: "2020-08-28 BikeLightComputer Rev 1"
- board text added: "Antenna"
- board text added: "Blue"
- board text added: "Green"
- board text added: "Off / On"
- board text added: "RX TX GND 3v3 Bluetooth LE"
- board text added: "Red"
- board text added: "http://douglas.malnati.com"
